File: lora1276Breakout.kicad_pcb (KiCad board)
At the start: 2 copper layers, 39.4 x 27.9 mm, 9 parts, among them J1 Conn_01x10_Male, U1 Lora1276_V2.0

Commit message: Adjust ant. track-width
Routing:
- net Net-(J2-Pad1): track 16.1 -> 18.2 mm
Changed lines of the file:
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@@
   (via (at 168.656 88.9) (size 0.8) (drill 0.4) (layers F.Cu B.Cu) (net 2))
   (segment (start 165.849906 87.394381) (end 167.150381 87.394381) (width 0.25) (layer F.Cu) (net 2))
-  (segment (start 167.150381 87.394381) (end 168.656 88.9) (width 0.25) (layer F.Cu) (net 2))
+  (segment (start 167.150381 87.394381) (end 168.656 88.9) (width 0.5) (layer F.Cu) (net 2))
   (segment (start 142.315619 100.254381) (end 142.24 100.33) (width 0.25) (layer F.Cu) (net 3))
   (segment (start 150.049906 100.254381) (end 142.315619 100.254381) (width 0.25) (layer F.Cu) (net 3))
@@
   (segment (start 146.558 85.768) (end 143.34 82.55) (width 0.25) (layer F.Cu) (net 10))
   (segment (start 146.558 88.646) (end 146.558 85.768) (width 0.25) (layer F.Cu) (net 10))
-  (segment (start 165.849906 85.894381) (end 168.952381 85.894381) (width 0.25) (layer F.Cu) (net 11))
-  (segment (start 168.952381 85.894381) (end 169.926 86.868) (width 0.25) (layer F.Cu) (net 11))
-  (segment (start 173.611 93.726) (end 175.006 93.726) (width 0.25) (layer F.Cu) (net 11))
-  (segment (start 169.926 86.868) (end 169.926 90.041) (width 0.25) (layer F.Cu) (net 11))
-  (via (at 171.704 91.819) (size 0.8) (drill 0.4) (layers F.Cu B.Cu) (net 11))
-  (segment (start 172.212 92.327) (end 171.704 91.819) (width 0.25) (layer B.Cu) (net 11))
-  (segment (start 172.212 93.472) (end 172.212 92.327) (width 0.25) (layer B.Cu) (net 11))
-  (segment (start 169.926 90.041) (end 171.704 91.819) (width 0.25) (layer F.Cu) (net 11))
-  (segment (start 171.704 91.819) (end 173.611 93.726) (width 0.25) (layer F.Cu) (net 11))
+  (segment (start 165.849906 85.894381) (end 168.952381 85.894381) (width 0.5) (layer F.Cu) (net 11))
+  (segment (start 168.952381 85.894381) (end 169.926 86.868) (width 0.5) (layer F.Cu) (net 11))
+  (segment (start 169.926 86.868) (end 169.926 90.041) (width 0.5) (layer F.Cu) (net 11))
+  (via (at 170.18 93.472) (size 0.8) (drill 0.4) (layers F.Cu B.Cu) (net 11))
+  (segment (start 169.926 90.041) (end 169.926 93.218) (width 0.5) (layer F.Cu) (net 11))
+  (segment (start 169.926 93.218) (end 170.18 93.472) (width 0.5) (layer F.Cu) (net 11))
+  (segment (start 170.18 93.472) (end 172.212 93.472) (width 0.5) (layer B.Cu) (net 11))
+  (segment (start 174.752 93.472) (end 175.006 93.726) (width 0.25) (layer F.Cu) (net 11))
+  (segment (start 170.18 93.472) (end 174.752 93.472) (width 0.5) (layer F.Cu) (net 11))
   (zone (net 1) (net_name +3V3) (layer F.Cu) (hatch edge 0.508)
     (connect_pads (clearance 0.508))
